Commit message: tried fixing some geometries

File: src/open_manipulator_p/open_manipulator_p_description/urdf/open_manipulator_p_with_flashlight.urdf.xacro (robot description, xacro)
@@ -257,5 +257,6 @@
       <origin xyz="0 0 0.05" rpy="0 0 0"/> <!-- Cylinder center -->
       <geometry>
-        <cylinder radius="0.02" length="0.1"/>
+        <!-- <cylinder radius="0.02" length="0.1"/> -->
+          <mesh filename="package://open_manipulator_p_description/meshes/cylinder.stl" scale="0.01 0.01 0.01"/>
       </geometry>
       <material name="blue"/>
@@ -264,5 +265,6 @@
       <origin xyz="0 0 0.05" rpy="0 0 0"/>
       <geometry>
-        <cylinder radius="0.02" length="0.1"/>
+        <!-- <cylinder radius="0.02" length="0.1"/> -->
+        <mesh filename="package://open_manipulator_p_description/meshes/cylinder.stl" scale="0.01 0.01 0.01"/>
       </geometry>
     </collision>
@@ -272,5 +274,6 @@
     <parent link="end_link"/> <!-- Replace with your robot’s last link if different -->
     <child link="flashlight_link"/>
-    <origin xyz="0.0 0.0 0.0" rpy="0 1.57 0"/>
+    <!-- <origin xyz="0.0 0.0 0.0" rpy="0 1.57 0"/> -->
+    <origin xyz="0.0 0.0 0.0" rpy="0 0 0"/>
   </joint>
   <link name="lightbeam_link">
@@ -279,6 +282,5 @@
       <origin xyz="0 0 0" rpy="0 0 0"/> <!-- cone starts after cylinder -->
       <geometry>
-        <mesh filename="package://open_manipulator_p_description/meshes/cone.stl" scale="0.01 0.01 0.01"/>
-        <!-- <cylinder radius="0.2" length="1.0"/> -->
+        <mesh filename="package://open_manipulator_p_description/meshes/new_cone.stl" scale="0.01 0.01 0.01"/>
       </geometry>
       <material name="light_beam"/>
@@ -296,5 +298,5 @@
     <parent link="flashlight_link"/> <!-- Replace with your robot’s last link if different -->
     <child link="lightbeam_link"/>
-    <origin xyz="0.0 0.0 1.1" rpy="3.1415 0 0"/>
+    <origin xyz="0.0 0.0 0.1" rpy="0 0 0"/>
   </joint>
 </robot>

Commit message: finished flashlight visualization

File: src/open_manipulator_p/open_manipulator_p_description/urdf/open_manipulator_p_with_flashlight.urdf.xacro (robot description, xacro)
@@ -255,16 +255,14 @@
   <link name="flashlight_link">
     <visual>
-      <origin xyz="0 0 0.05" rpy="0 0 0"/> <!-- Cylinder center -->
-      <geometry>
-        <!-- <cylinder radius="0.02" length="0.1"/> -->
-          <mesh filename="package://open_manipulator_p_description/meshes/cylinder.stl" scale="0.01 0.01 0.01"/>
+      <origin xyz="0.05 0 0" rpy="0 0 0"/> <!-- Cylinder center -->
+      <geometry>
+          <mesh filename="package://open_manipulator_p_description/meshes/cylinder.stl" scale="1.0 1.0 1.0"/>
       </geometry>
       <material name="blue"/>
     </visual>
     <collision>
-      <origin xyz="0 0 0.05" rpy="0 0 0"/>
-      <geometry>
-        <!-- <cylinder radius="0.02" length="0.1"/> -->
-        <mesh filename="package://open_manipulator_p_description/meshes/cylinder.stl" scale="0.01 0.01 0.01"/>
+      <origin xyz="0.05 0 0" rpy="0 0 0"/>
+      <geometry>
+        <mesh filename="package://open_manipulator_p_description/meshes/cylinder.stl" scale="1.0 1.0 1.0"/>
       </geometry>
     </collision>
@@ -274,5 +272,4 @@
     <parent link="end_link"/> <!-- Replace with your robot’s last link if different -->
     <child link="flashlight_link"/>
-    <!-- <origin xyz="0.0 0.0 0.0" rpy="0 1.57 0"/> -->
     <origin xyz="0.0 0.0 0.0" rpy="0 0 0"/>
   </joint>
@@ -282,5 +279,5 @@
       <origin xyz="0 0 0" rpy="0 0 0"/> <!-- cone starts after cylinder -->
       <geometry>
-        <mesh filename="package://open_manipulator_p_description/meshes/new_cone.stl" scale="0.01 0.01 0.01"/>
+        <mesh filename="package://open_manipulator_p_description/meshes/cone.stl" scale="0.01 0.01 0.01"/>
       </geometry>
       <material name="light_beam"/>
@@ -298,5 +295,5 @@
     <parent link="flashlight_link"/> <!-- Replace with your robot’s last link if different -->
     <child link="lightbeam_link"/>
-    <origin xyz="0.0 0.0 0.1" rpy="0 0 0"/>
+    <origin xyz="0.08 0.0 0.0" rpy="0 0 0"/>
   </joint>
 </robot>
